File: KiCad/_autosave-rubiks-cub.kicad_sch (KiCad schematic)
At the start: 42 parts, among them J1 USB_B_Mini, J10 Conn_01x03_Pin, J11 Conn_01x03_Pin, J2 Conn_01x04_Pin, J3 Conn_01x04_Pin, J4 Conn_01x04_Pin, J5 Jack-DC, J6 Conn_01x04_Pin, J7 Conn_01x03_Pin, J8 Conn_01x03_Pin, J9 Conn_01x04_Pin, SW1 SW_SPDT, SW2 SW_Push, U1 STM32F401RETx, U2 AMS1117-3.3, Y1 16MHz

Commit message: schematic done
Connections:
- net +3.3VA: now also FB1.2, U1.13 (VREF+); no longer FB1.1
- net at C8.1: now also FB1.1; no longer FB1.2
- no-connect marks 39 -> 38
Other:
- note added: "Crystal oscillator"
- moved on the sheet: C10, C11, C6, C7, C8, FB1, Y1
