File: KiCad/rubiks-cub.kicad_sch (KiCad schematic)
At the start: 18 parts, among them J1 USB_B_Mini, SW1 SW_SPDT, U1 STM32F401RETx, Y1 16MHz

Commit message: KiCad
Parts:
- added J2: Conn_01x04_Pin, symbol Connector:Conn_01x04_Pin
Connections:
- net +3.3V: now also J2.1 (Pin_1)
- net GND: now also J2.4 (Pin_4)
- net SW_DIO: now reaches U1.46 (PA13)
- net SW_DIO: now also J2.2 (Pin_2)
- net SM_CLK: now reaches U1.49 (PA14)
- net SM_CLK: now also J2.3 (Pin_3)

Commit message: -
Parts:
- added R3: 1k5, symbol Device:R
Changed lines of the file:
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@@
+	)
+	(symbol
+		(lib_id "Device:R")
+		(at 171.45 63.5 0)
+		(unit 1)
+		(exclude_from_sim no)
+		(in_bom yes)
+		(on_board yes)
+		(dnp no)
+		(fields_autoplaced yes)
+		(property "Reference" "R3"
+			(at 173.99 62.2299 0)
+			(effects
+				(font
+					(size 1.27 1.27)
+				)
+				(justify left)
+			)
+		)
+		(property "Value" "1k5"
+			(at 173.99 64.7699 0)
+			(effects
+				(font
+					(size 1.27 1.27)
+				)
+				(justify left)
+			)
+		)
+		(property "Footprint" ""
+			(at 169.672 63.5 90)
+			(effects
+				(font
+					(size 1.27 1.27)
+				)
+				(hide yes)
+			)
+		)
+		(property "Datasheet" "~"
+			(at 171.45 63.5 0)
+			(effects
+				(font
+					(size 1.27 1.27)
+				)
+				(hide yes)
+			)
+		)
+		(property "Description" "Resistor"
+			(at 171.45 63.5 0)
+			(effects
+				(font
+					(size 1.27 1.27)
+				)
+				(hide yes)
+			)
+		)
+		(pin "2"
+		)
+		(pin "1"
+		)
+		(instances
+			(project "rubiks-cub"
+				(path "/0d0eb51a-0624-4b1b-872b-cd4472588f67"
+					(reference "R3")
+					(unit 1)
+				)
+			)
+		)
 	)
 	(symbol

Commit message: demo pcb schematic done
Parts:
- added C12, C13: 22u, symbol Device:C
- added D1: RED, symbol Device:LED
- added J3, J4: Conn_01x04_Pin, symbol Connector:Conn_01x04_Pin
- added R4, R6: 1k5, symbol Device:R
- added U2: AMS1117-3.3, Package_TO_SOT_SMD:SOT-223-3_TabPin2, symbol Regulator_Linear:AMS1117-3.3
Connections:
- net +3.3V: now also R3.1, C13.1, D1.2 (A), J3.1 (Pin_1), J4.1 (Pin_1), R6.1, U2.2 (VO)
- net GND: now also C12.2, C13.2, J3.4 (Pin_4), J4.4 (Pin_4), R4.2, U2.1 (GND)
- net VBUS: now also C12.1, U2.3 (VI)
- net USART1_TX: now reaches U1.58 (PB6)
- net USART1_TX: now also J3.2 (Pin_2)
- net USART1_RX: now reaches U1.59 (PB7)
- net USART1_RX: now also J3.3 (Pin_3)
- net I2C_SCL: now reaches U1.61 (PB8)
- net I2C_SCL: now also R3.2, J4.2 (Pin_2)
- net I2C_SDA: now reaches U1.62 (PB9)
- net I2C_SDA: now also J4.3 (Pin_3), R6.2
- new net: D1.1 (K), R4.1
- no-connect marks 2 -> 43
Other:
- note added: "Microcontroller and USB"
- note added: "Power Supply"
- note added: "Rubik's cube: Demo PCB"
- company: (none) -> Wilgot Wardell
- title: Rubiks Cube Robot -> Rubiks Cube Robot: Demo
- moved on the sheet: C1, C10, C11, C2, C3, C4, C5, C6, C7, C8, C9, FB1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
