File: KiCad/rubiks-cub.kicad_sch (KiCad schematic)
At the start: 28 parts, among them J1 USB_B_Mini, J2 Conn_01x04_Pin, J3 Conn_01x04_Pin, J4 Conn_01x04_Pin, SW1 SW_SPDT, U1 STM32F401RETx, U2 AMS1117-3.3, Y1 16MHz

Commit message: added extra components
Parts:
- added A1: Pololu_Breakout_A4988, Module:Pololu_Breakout-16_15.2x20.3mm, symbol Driver_Motor:Pololu_Breakout_A4988
- added C14: 470u, symbol Device:C
- added C15: 100p, symbol Device:C
- added D2: SS34, Diode_SMD:D_SMA, symbol Diode:SS34
- added J5: Jack-DC, symbol Connector:Jack-DC
- added J6: Conn_01x04_Pin, symbol Connector:Conn_01x04_Pin
- added J7, J8: Conn_01x08_Socket, symbol Connector:Conn_01x08_Socket
Connections:
- net +3.3V: now also A1.2 (VDD)
- net GND: now also A1.1 (GND), A1.7 (GND), C14.2, J5.2, J6.1 (Pin_1), J6.3 (Pin_3)
- net VBUS: no longer C12.1, U2.3 (VI)
- new net: A1.13 (~{RESET}), A1.14 (~{SLEEP})
- new net: A1.8 (VMOT), C15.2
- new net: C14.1, D2.1 (K)
- new net +12: D2.2 (A), J5.1, J6.4 (Pin_4)
- new net +12V: C15.1
- new net +5V_PWR: C12.1, J6.2 (Pin_2), U2.3 (VI)
- no-connect marks 44 -> 47
Other:
- note added: "Connect external LM2596 buck converter"
- note removed: "Power Supply"
- moved on the sheet: C1, C10, C11, C12, C13, C2, C3, C4, C5, C6, C7, C8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

Commit message: -
Parts:
- removed J7, J8: Conn_01x08_Socket, symbol Connector:Conn_01x08_Socket
- added C16: 100n, symbol Device:C
- added C17: 4.7u, symbol Device:C
- added J10, J11, J7, J8: Conn_01x03_Pin, symbol Connector:Conn_01x03_Pin
- added J9: Conn_01x04_Pin, symbol Connector:Conn_01x04_Pin
- C15: value 100p -> 100u
Connections:
- net +12: no longer J6.4 (Pin_4)
- net +3.3V: now also U1.64 (VDD), C16.1
- net GND: now also C16.2, C17.2, J10.3 (Pin_3), J11.3 (Pin_3), J7.3 (Pin_3), J8.3 (Pin_3)
- net enable_sm: now reaches U1.10 (PC2)
- net enable_sm: now also A1.9 (~{ENABLE})
- net at U1.15 (PA1): now also J11.1 (Pin_1)
- net at U1.16 (PA2): now also J7.1 (Pin_1)
- net at U1.17 (PA3): now also J8.1 (Pin_1)
- net at U1.20 (PA4): now also J10.1 (Pin_1)
- net at U1.30 (VCAP1): now also C17.1
- net dir_sm: now reaches U1.8 (PC0)
- net dir_sm: now also A1.16 (DIR)
- net step_sm: now reaches U1.9 (PC1)
- net step_sm: now also A1.15 (STEP)
- net at A1.3 (1B): now also J9.1 (Pin_1)
- net at A1.4 (1A): now also J9.2 (Pin_2)
- net at A1.5 (2A): now also J9.3 (Pin_3)
- net at A1.6 (2B): now also J9.4 (Pin_4)
- net IN+: now reaches C14.1, D2.1 (K)
- net IN+: now also J6.4 (Pin_4)
- net +5V_PWR renamed +5V
- net +5V: now also J10.2 (Pin_2), J11.2 (Pin_2), J7.2 (Pin_2), J8.2 (Pin_2)
- no-connect marks 47 -> 39
Other:
- note added: "A4988 motor driver for the NEMA 14 stepper motor"
- note added: "Powersupply"
- note added: "converts to +3.3V for MCU"
- note added: "converts to +5V for servos"
- moved on the sheet: A1, C1, C10, C11, C12, C13, C14, C15, C2, C3, C4, C5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
