File: KiCad/rubiks-cub.kicad_sch (KiCad schematic)
At the start: 42 parts, among them J1 USB_B_Mini, J10 Conn_01x03_Pin, J11 Conn_01x03_Pin, J2 Conn_01x04_Pin, J3 Conn_01x04_Pin, J4 Conn_01x04_Pin, J5 Jack-DC, J6 Conn_01x04_Pin, J7 Conn_01x03_Pin, J8 Conn_01x03_Pin, J9 Conn_01x04_Pin, SW1 SW_SPDT, SW2 SW_Push, U1 STM32F401RETx, U2 AMS1117-3.3, Y1 16MHz

Commit message: -
Parts:
- added J12: Conn_01x03_Pin, symbol Connector:Conn_01x03_Pin
Connections:
- net +3.3VA: now also FB1.2, U1.13 (VREF+); no longer FB1.1
- net +5V: now also J12.2 (Pin_2)
- net GND: now also J12.3 (Pin_3)
- net USART1_RX: now also J3.2 (Pin_2); no longer J3.3 (Pin_3)
- net USART1_TX: now also J3.3 (Pin_3); no longer J3.2 (Pin_2)
- net at C8.1: now also FB1.1; no longer FB1.2
- net at U1.16 (PA2): no longer J7.1 (Pin_1)
- net at U1.17 (PA3): no longer J8.1 (Pin_1)
- net at U1.15 (PA1): no longer J11.1 (Pin_1)
- net at U1.20 (PA4): no longer J10.1 (Pin_1)
- net SERVO1: now reaches U1.21 (PA5)
- net SERVO1: now also J11.1 (Pin_1)
- net SERVO2: now reaches U1.22 (PA6)
- net SERVO2: now also J7.1 (Pin_1)
- net SERVO3: now reaches U1.23 (PA7)
- net SERVO3: now also J8.1 (Pin_1)
- net at U1.29 (PB10): now also J12.1 (Pin_1)
- net SERVO4: now reaches U1.42 (PA9)
- net SERVO4: now also J10.1 (Pin_1)
- no-connect marks 39 -> 37
Other:
- note added: "Color sensor port"
- note added: "Connect TCS34725 sensor"
- note added: "Crystal oscillator"
- note added: "Robot arm connectors"
- note added: "ST-LINK programmer"
- note added: "UART communication"
- moved on the sheet: A1, C1, C10, C11, C12, C13, C14, C15, C16, C17, C2, C3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

Commit message: -
Connections:
- net +12V: now also A1.8 (VMOT), C15.2; no longer C15.1
- net GND: now also C15.1
- net SERVO5: now reaches J12.1 (Pin_1), U1.29 (PB10)
- net SM_CLK renamed SW_CLK
Other:
- moved on the sheet: C15, C17

Commit message: -
Connections:
- net IN+ is gone; now on net +12V: C14.1, D2.1 (K), J6.4 (Pin_4)
Other:
- note added: "Connect NEMA17 stepper motor"
Changed lines of the file:
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@@
 	)
 	(rectangle
-		(start 127 41.91)
+		(start 127 43.18)
 		(end 295.91 191.77)
 		(stroke
@@
 	(text "Microcontroller and USB\n"
 		(exclude_from_sim no)
-		(at 148.082 44.958 0)
+		(at 147.066 39.37 0)
 		(effects
 			(font
@@
 		)
 	)
+	(text "Connect NEMA17\nstepper motor\n"
+		(exclude_from_sim no)
+		(at 169.672 176.022 0)
+		(effects
+			(font
+				(size 1 1)
+			)
+		)
+	)
 	(junction
 		(at 161.29 130.81)
@@
 	(wire
 		(pts
-			(xy 167.64 204.47) (xy 167.64 219.71)
-		)
-		(stroke
-			(width 0)
-			(type default)
-		)
-	)
-	(wire
-		(pts
 			(xy 247.65 120.65) (xy 247.65 121.92)
 		)
@@
 	(wire
 		(pts
+			(xy 167.64 219.71) (xy 173.99 219.71)
+		)
+		(stroke
+			(width 0)
+			(type default)
+		)
+	)
+	(wire
+		(pts
 			(xy 171.45 209.55) (xy 177.8 209.55)
 		)
@@
 	(wire
 		(pts
+			(xy 167.64 204.47) (xy 167.64 219.71)
+		)
+		(stroke
+			(width 0)
+			(type default)
+		)
+	)
+	(wire
+		(pts
 			(xy 139.7 158.75) (xy 135.89 158.75)
 		)
@@
 					(unit 1)
 				)
+			)
+		)
+	)
+	(symbol
+		(lib_id "power:+3.3V")
+		(at 173.99 219.71 0)
+		(unit 1)
+		(exclude_from_sim no)
+		(in_bom yes)
+		(on_board yes)
+		(dnp no)
+		(property "Reference" "#PWR034"
+			(at 173.99 223.52 0)
+			(effects
+				(font
+					(size 1.27 1.27)
+				)
+				(hide yes)
+			)
+		)
+		(property "Value" "+12V"
+			(at 173.99 216.154 0)
+			(effects
+				(font
+					(size 1.27 1.27)
+				)
+			)
+		)
+		(property "Footprint" ""
+			(at 173.99 219.71 0)
+			(effects
+				(font
+					(size 1.27 1.27)
+				)
+				(hide yes)
+			)
+		)
+		(property "Datasheet" ""
+			(at 173.99 219.71 0)
+			(effects
+				(font
+					(size 1.27 1.27)
+				)
+				(hide yes)
+			)
+		)
+		(property "Description" "Power symbol creates a global label with name \"+3.3V\""
+			(at 173.99 219.71 0)
+			(effects
+				(font
+					(size 1.27 1.27)
+				)
+				(hide yes)
+			)
+		)
+		(pin "1"
+		)
+		(instances
+			(project "rubiks-cub"
+				(path "/0d0eb51a-0624-4b1b-872b-cd4472588f67"
+					(reference "#PWR034")
+					(unit 1)
+				)

Commit message: -
Parts:
- C1, C10, C11, C16, C2, C3, C4, C6, C7, C8, C9: footprint (none) -> Capacitor_SMD:C_0402_1005Metric
- C12, C13: footprint (none) -> Capacitor_SMD:C_0805_2012Metric
- C14, C15: footprint (none) -> Capacitor_THT:C_Radial_D8.0mm_H7.0mm_P3.50mm
- C17, C5: footprint (none) -> Capacitor_SMD:C_0603_1608Metric
- D1: footprint (none) -> LED_SMD:LED_0603_1608Metric
- FB1: footprint (none) -> Inductor_SMD:L_0603_1608Metric
- J1: footprint (none) -> Connector_USB:USB_Mini-B_Wuerth_65100516121_Horizontal
- J10, J11, J12, J7, J8: footprint (none) -> Connector_PinHeader_1.00mm:PinHeader_1x03_P1.00mm_Vertical
- J2, J3, J4, J6, J9: footprint (none) -> Connector_PinHeader_1.00mm:PinHeader_1x04_P1.00mm_Vertical
- J5: footprint (none) -> Connector_BarrelJack:BarrelJack_Horizontal
- R1, R2, R3, R4, R6: footprint (none) -> Resistor_SMD:R_0402_1005Metric
- SW1: footprint (none) -> Button_Switch_SMD:SW_SPDT_PCM12
- SW2: footprint (none) -> Button_Switch_THT:SW_PUSH_6mm
- Y1: footprint (none) -> Crystal:Crystal_SMD_3225-4Pin_3.2x2.5mm
Connections:
- net +3.3V: now also C8.1, FB1.1
Other:
- moved on the sheet: C6, C7, C8, FB1

Commit message: -
Connections:
- net +12 is gone; now on net +12V: D2.2 (A), J5.1
Changed lines of the file:
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@@
 		)
 	)
-	(label "+12"
+	(label "+12V"
 		(at 156.21 219.71 180)
 		(effects

Commit message: -
Parts:
- removed J6: Conn_01x04_Pin, Connector_PinHeader_1.00mm:PinHeader_1x04_P1.00mm_Vertical, symbol Connector:Conn_01x04_Pin
- added J13, J14, J15, J6: Conn_01x01_Pin, Connector_PinHeader_2.54mm:PinHeader_1x01_P2.54mm_Vertical, symbol Connector:Conn_01x01_Pin
Connections:
- net +12V: now also J6.1 (Pin_1)
- net +5V: now also J14.1 (Pin_1)
- net GND: now also J13.1 (Pin_1), J15.1 (Pin_1)
- net VCAP: now reaches C17.1, U1.30 (VCAP1)
Other:
- note added: "A4988 motor driver for the NEMA 17 stepper motor"
- note removed: "A4988 motor driver for the NEMA 14 stepper motor"
Changed lines of the file:
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@@
 		)
 	)
-	(text "A4988 motor driver for \nthe NEMA 14 stepper motor "
+	(text "A4988 motor driver for \nthe NEMA 17 stepper motor "
 		(exclude_from_sim no)
 		(at 143.002 141.478 0)
@@
 	(text "Connect external \nLM2596 buck converter"
 		(exclude_from_sim no)
-		(at 138.43 202.184 0)
+		(at 140.716 200.66 0)
 		(effects
 			(font
@@
 	(wire
 		(pts
-			(xy 167.64 219.71) (xy 173.99 219.71)
+			(xy 167.64 219.71) (xy 171.45 219.71)
 		)
 		(stroke
@@
 		)
 	)
+	(label "VCAP"
+		(at 196.85 143.51 90)
+		(effects
+			(font
+				(size 1.27 1.27)
+			)
+			(justify left bottom)
+		)
+	)
 	(label "HSE_OUT"
 		(at 189.23 90.17 0)
@@
 	)
 	(symbol
+		(lib_id "Connector:Conn_01x01_Pin")
+		(at 147.32 209.55 0)
+		(unit 1)
+		(exclude_from_sim no)
+		(in_bom yes)
+		(on_board yes)
+		(dnp no)
+		(property "Reference" "J14"
+			(at 143.764 209.296 0)
+			(effects
+				(font
+					(size 1.27 1.27)
+				)
+			)
+		)
+		(property "Value" "Conn_01x01_Pin"
+			(at 112.268 207.264 0)
+			(effects
+				(font
+					(size 1.27 1.27)
+				)
+				(hide yes)
+			)
+		)
+		(property "Footprint" "Connector_PinHeader_2.54mm:PinHeader_1x01_P2.54mm_Vertical"
+			(at 147.32 209.55 0)
+			(effects
+				(font
+					(size 1.27 1.27)
+				)
+				(hide yes)
+			)
+		)
+		(property "Datasheet" "~"
+			(at 147.32 209.55 0)
+			(effects
+				(font
+					(size 1.27 1.27)
+				)
+				(hide yes)
+			)
+		)
+		(property "Description" "Generic connector, single row, 01x01, script generated"
+			(at 147.32 209.55 0)
+			(effects
+				(font
+					(size 1.27 1.27)
+				)
+				(hide yes)
+			)
+		)
+		(pin "1"
+		)
+		(instances
+			(project "rubiks-cub"
+				(path "/0d0eb51a-0624-4b1b-872b-cd4472588f67"
+					(reference "J14")
+					(unit 1)
+				)
+			)
+		)
+	)
+	(symbol
 		(lib_id "Device:C")
 		(at 148.59 113.03 0)
@@
 		)
 		(property "Value" "PWR_FLAG"
-			(at 147.066 215.646 0)
+			(at 151.384 216.408 0)
 			(effects
 				(font
@@
 	)
 	(symbol
+		(lib_id "Connector:Conn_01x01_Pin")
+		(at 147.32 207.01 0)
+		(unit 1)
+		(exclude_from_sim no)
+		(in_bom yes)
+		(on_board yes)
+		(dnp no)
+		(property "Reference" "J13"
+			(at 143.764 206.756 0)
+			(effects
+				(font
+					(size 1.27 1.27)
+				)
+			)
+		)
+		(property "Value" "Conn_01x01_Pin"
+			(at 112.268 204.724 0)
+			(effects
+				(font
+					(size 1.27 1.27)
+				)
+				(hide yes)
+			)
+		)
+		(property "Footprint" "Connector_PinHeader_2.54mm:PinHeader_1x01_P2.54mm_Vertical"
+			(at 147.32 207.01 0)
+			(effects
+				(font
+					(size 1.27 1.27)
+				)
+				(hide yes)
+			)
+		)
+		(property "Datasheet" "~"
+			(at 147.32 207.01 0)
+			(effects
+				(font
+					(size 1.27 1.27)
+				)
+				(hide yes)
+			)
+		)
+		(property "Description" "Generic connector, single row, 01x01, script generated"
+			(at 147.32 207.01 0)
+			(effects
+				(font
+					(size 1.27 1.27)
+				)
+				(hide yes)
+			)
+		)
+		(pin "1"
+		)
+		(instances
+			(project "rubiks-cub"
+				(path "/0d0eb51a-0624-4b1b-872b-cd4472588f67"
+					(reference "J13")
+					(unit 1)
+				)
+			)
+		)
+	)
+	(symbol
 		(lib_id "Connector:Conn_01x04_Pin")
 		(at 280.67 123.19 0)
@@
 	)
 	(symbol
+		(lib_id "Connector:Conn_01x01_Pin")
+		(at 147.32 212.09 0)
+		(unit 1)
+		(exclude_from_sim no)
+		(in_bom yes)
+		(on_board yes)
+		(dnp no)
+		(property "Reference" "J15"
+			(at 143.764 211.836 0)
+			(effects
+				(font
+					(size 1.27 1.27)
+				)
+			)
+		)
+		(property "Value" "Conn_01x01_Pin"
+			(at 112.268 209.804 0)
+			(effects
+				(font
+					(size 1.27 1.27)
+				)
+				(hide yes)
+			)
+		)
+		(property "Footprint" "Connector_PinHeader_2.54mm:PinHeader_1x01_P2.54mm_Vertical"
+			(at 147.32 212.09 0)
+			(effects
+				(font
+					(size 1.27 1.27)
+				)
+				(hide yes)
+			)
+		)
+		(property "Datasheet" "~"
+			(at 147.32 212.09 0)
+			(effects
+				(font
+					(size 1.27 1.27)
+				)
+				(hide yes)
+			)
+		)
+		(property "Description" "Generic connector, single row, 01x01, script generated"
+			(at 147.32 212.09 0)
+			(effects
+				(font
+					(size 1.27 1.27)
+				)
+				(hide yes)
+			)
+		)
+		(pin "1"
+		)
+		(instances
+			(project "rubiks-cub"
+				(path "/0d0eb51a-0624-4b1b-872b-cd4472588f67"
+					(reference "J15")
+					(unit 1)
+				)
+			)
+		)
+	)
+	(symbol
 		(lib_id "Switch:SW_SPDT")
 		(at 170.18 77.47 180)
@@
 	)
 	(symbol
-		(lib_id "Connector:Conn_01x04_Pin")
-		(at 147.32 209.55 0)
-		(mirror x)
-		(unit 1)
-		(exclude_from_sim no)
-		(in_bom yes)
-		(on_board yes)
-		(dnp no)
-		(fields_autoplaced yes)
-		(property "Reference" "J6"
-			(at 146.05 207.0099 0)
-			(effects
-				(font
-					(size 1.27 1.27)
-				)
-				(justify right)
-			)
-		)
-		(property "Value" "Conn_01x04_Pin"
-			(at 146.05 209.5499 0)
-			(effects
-				(font
-					(size 1.27 1.27)
-				)
-				(justify right)
-			)
-		)
-		(property "Footprint" "Connector_PinHeader_1.00mm:PinHeader_1x04_P1.00mm_Vertical"
-			(at 147.32 209.55 0)
-			(effects
-				(font
-					(size 1.27 1.27)
-				)
-				(hide yes)
-			)
-		)
-		(property "Datasheet" "~"
-			(at 147.32 209.55 0)
-			(effects
-				(font
-					(size 1.27 1.27)
-				)
-				(hide yes)
-			)
-		)
-		(property "Description" "Generic connector, single row, 01x04, script generated"
-			(at 147.32 209.55 0)
-			(effects
-				(font
-					(size 1.27 1.27)
-				)
-				(hide yes)
-			)
-		)
-		(pin "4"
-		)
-		(pin "3"
-		)
-		(pin "1"
-		)
-		(pin "2"
-		)
-		(instances
-			(project "rubiks-cub"
-				(path "/0d0eb51a-0624-4b1b-872b-cd4472588f67"
-					(reference "J6")
-					(unit 1)
-				)
-			)
-		)
-	)
-	(symbol
 		(lib_id "power:GND")
 		(at 140.97 123.19 0)
@@
 	(symbol
 		(lib_id "power:+3.3V")
-		(at 173.99 219.71 0)
+		(at 171.45 219.71 0)
 		(unit 1)
 		(exclude_from_sim no)
@@
 		(dnp no)
 		(property "Reference" "#PWR034"
-			(at 173.99 223.52 0)
+			(at 171.45 223.52 0)
 			(effects
 				(font
@@
 		)
 		(property "Value" "+12V"
-			(at 173.99 216.154 0)
+			(at 171.45 216.154 0)
 			(effects
 				(font
@@
 		)
 		(property "Footprint" ""
-			(at 173.99 219.71 0)
+			(at 171.45 219.71 0)
 			(effects
 				(font
@@
 		)
 		(property "Datasheet" ""
-			(at 173.99 219.71 0)
+			(at 171.45 219.71 0)
 			(effects
 				(font
@@
 		)
 		(property "Description" "Power symbol creates a global label with name \"+3.3V\""
-			(at 173.99 219.71 0)
+			(at 171.45 219.71 0)
 			(effects
 				(font
@@
 					(unit 1)
 				)
+			)
+		)
+	)
+	(symbol
+		(lib_id "Connector:Conn_01x01_Pin")
+		(at 147.32 204.47 0)
+		(unit 1)
+		(exclude_from_sim no)
+		(in_bom yes)
+		(on_board yes)
+		(dnp no)
+		(property "Reference" "J6"
+			(at 143.764 204.216 0)
+			(effects
+				(font
+					(size 1.27 1.27)
+				)
+			)
+		)
+		(property "Value" "Conn_01x01_Pin"
+			(at 112.268 202.184 0)
+			(effects
+				(font
+					(size 1.27 1.27)
+				)
+				(hide yes)
+			)
+		)
+		(property "Footprint" "Connector_PinHeader_2.54mm:PinHeader_1x01_P2.54mm_Vertical"
+			(at 147.32 204.47 0)
+			(effects
+				(font
+					(size 1.27 1.27)
+				)
+				(hide yes)
+			)
+		)
+		(property "Datasheet" "~"
+			(at 147.32 204.47 0)
+			(effects
+				(font
+					(size 1.27 1.27)
+				)
+				(hide yes)
+			)
+		)
+		(property "Description" "Generic connector, single row, 01x01, script generated"
+			(at 147.32 204.47 0)
+			(effects
+				(font
+					(size 1.27 1.27)
+				)
+				(hide yes)
+			)
+		)
+		(pin "1"
+		)
+		(instances
+			(project "rubiks-cub"
+				(path "/0d0eb51a-0624-4b1b-872b-cd4472588f67"
+					(reference "J6")
+					(unit 1)
+				)

Commit message: pcb design
Parts:
- added H1, H2, H3, H4: MountingHole, MountingHole:MountingHole_2.2mm_M2, symbol Mechanical:MountingHole
Other:
- note added: "M2 2.2mm"
- note added: "Mounting holes"

Commit message: -
Connections:
- net +12V: no longer D2.2 (A), J5.1
- new net DC_IN: D2.2 (A), J5.1
Changed lines of the file:
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@@
 		)
 	)
-	(label "+12V"
+	(label "DC_IN"
 		(at 156.21 219.71 180)
 		(effects
 			(font
-				(size 1.27 1.27)
+				(size 1 1)
 			)
 			(justify right bottom)
