File: KiCad/rubiks-cub.kicad_pcb (KiCad board)
At the start: 2 copper layers, 43 parts, among them J1 USB_B_Mini, J10 Conn_01x03_Pin, J11 Conn_01x03_Pin, J12 Conn_01x03_Pin, J2 Conn_01x04_Pin, J3 Conn_01x04_Pin, J4 Conn_01x04_Pin, J5 Jack-DC, J6 Conn_01x04_Pin, J7 Conn_01x03_Pin, J8 Conn_01x03_Pin, J9 Conn_01x04_Pin, SW1 SW_SPDT, SW2 SW_Push, U1 STM32F401RETx, U2 AMS1117-3.3, Y1 16MHz

Commit message: -
Parts:
- moved C5 118.2 mm to (180.4, 117.8)
- moved R4 118.0 mm to (175.0, 132.2)
- moved C17 113.1 mm to (175.0, 121.6), turned to -90 degrees
- moved R3 112.2 mm to (174.8, 103.8)
- moved C13 112.0 mm to (172.8, 135.8)
- moved C14 110.4 mm to (155.6, 138.4)
- moved R6 109.6 mm to (172.5, 103.8), turned to 180 degrees
- moved C12 108.8 mm to (168.8, 135.8)
- moved R1 107.9 mm to (169.8, 105.0), turned to 90 degrees
- moved J3 106.4 mm to (180.2, 101.0), turned to -90 degrees
- moved D1 103.5 mm to (171.8, 132.1), turned to 180 degrees
- moved J10 103.4 mm to (179.5, 113.0), turned to 90 degrees
- moved J7 103.2 mm to (170.2, 124.8)
- moved J8 102.3 mm to (172.6, 124.8)
- moved A1 101.3 mm to (144.7, 113.6)
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Connections:
- D2 pad 2: /+12 -> +12V
- J5 pad 1: /+12 -> +12V

Commit message: -
Parts:
- added J13: Conn_01x01_Pin, Connector_PinHeader_2.54mm:PinHeader_1x01_P2.54mm_Vertical, F.Cu at (104.4, 128.4)
- added J14: Conn_01x01_Pin, Connector_PinHeader_2.54mm:PinHeader_1x01_P2.54mm_Vertical, F.Cu at (104.4, 114.6)
- added J15: Conn_01x01_Pin, Connector_PinHeader_2.54mm:PinHeader_1x01_P2.54mm_Vertical, F.Cu at (63.4, 128.4)
- J6: value Conn_01x04_Pin -> Conn_01x01_Pin; footprint Connector_PinHeader_1.00mm:PinHeader_1x04_P1.00mm_Vertical -> Connector_PinHeader_2.54mm:PinHeader_1x01_P2.54mm_Vertical
- moved J6 103.2 mm to (63.4, 114.6), turned to 0 degrees
- moved J5 71.6 mm to (79.8, 137.6)
- moved D2 71.5 mm to (74.0, 134.6), turned to 180 degrees
- moved R4 67.2 mm to (107.8, 132.6), turned to -90 degrees
- moved D1 66.4 mm to (105.4, 132.8)
- moved U2 66.0 mm to (104.8, 140.8)
- moved C12 66.0 mm to (102.8, 135.2)
- moved C13 66.0 mm to (106.8, 135.2)
- moved C14 64.0 mm to (91.6, 137.7), turned to -90 degrees
- moved C15 61.4 mm to (79.0, 106.4), turned to 180 degrees
- moved J4 58.3 mm to (117.0, 106.6), turned to 0 degrees
- moved J3 56.2 mm to (124.4, 107.6), turned to 0 degrees
- moved R3 54.8 mm to (120.4, 110.6), turned to -90 degrees
- moved R6 53.7 mm to (119.2, 110.6), turned to -90 degrees
- moved J1 52.9 mm to (138.4, 119.5)
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Connections:
- net Net-(U1-VCAP1) renamed /VCAP
- J6 pad 1: GND -> +12V

Commit message: pcb design
Parts:
- added H1: MountingHole, MountingHole:MountingHole_2.2mm_M2, F.Cu at (62.0, 95.0)
- added H2: MountingHole, MountingHole:MountingHole_2.2mm_M2, F.Cu at (142.0, 95.0)
- added H3: MountingHole, MountingHole:MountingHole_2.2mm_M2, F.Cu at (62.0, 145.0)
- added H4: MountingHole, MountingHole:MountingHole_2.2mm_M2, F.Cu at (142.0, 145.0)
- moved J9 19.3 mm to (77.5, 95.2), turned to 0 degrees
- moved J2 10.9 mm to (129.0, 99.5), turned to 0 degrees
- moved SW1 8.40 mm to (122.5, 94.0)
- moved J3 8.12 mm to (125.0, 99.5)
- moved J4 7.14 mm to (117.8, 99.5)
- moved D2 3.75 mm to (70.2, 134.6)
- moved C9 3.62 mm to (112.2, 97.4)
- moved R1 3.62 mm to (122.0, 107.0)
- moved SW2 3.62 mm to (109.8, 106.2)
- moved R3 3.62 mm to (120.8, 107.0)
- moved R6 3.62 mm to (119.6, 107.0)
- moved J5 3.60 mm to (80.0, 134.0)
- moved J7 2.49 mm to (119.8, 132.8)
- moved J11 2.49 mm to (117.2, 132.8)
- moved J12 2.29 mm to (127.4, 132.8)
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Other:
- board outline added: 86 x 56 mm
