File: KiCad/rubiks-cub.kicad_pcb (KiCad board)
At the start: 2 copper layers, 86 x 56 mm, 50 parts, among them J1 USB_B_Mini, J10 Conn_01x03_Pin, J11 Conn_01x03_Pin, J12 Conn_01x03_Pin, J13 Conn_01x01_Pin, J14 Conn_01x01_Pin, J15 Conn_01x01_Pin, J2 Conn_01x04_Pin, J3 Conn_01x04_Pin, J4 Conn_01x04_Pin, J5 Jack-DC, J6 Conn_01x01_Pin, J7 Conn_01x03_Pin, J8 Conn_01x03_Pin, J9 Conn_01x04_Pin, SW1 SW_SPDT, SW2 SW_Push, U1 STM32F401RETx, U2 AMS1117-3.3, Y1 16MHz

Commit message: -
Parts:
- moved C1 1.54 mm to (115.5, 114.2)
- moved C4 1.41 mm to (119.0, 111.0), turned to 0 degrees
- moved C3 1.20 mm to (130.0, 113.4)
- moved C2 0.75 mm to (127.6, 125.8), turned to -90 degrees
- moved C5 0.40 mm to (129.8, 124.0)
- moved FB1 0.11 mm to (116.6, 124.5)
Routing:
- net GND: track 0.00 -> 12.9 mm
- net +3.3V: track 0.00 -> 12.2 mm
- net /VCAP: track 0.00 -> 2.52 mm
- net +3.3VA: track 0.00 -> 1.85 mm
- added copper zone on B.Cu, net GND

Commit message: pcb progress
Parts:
- moved J9 18.8 mm to (96.2, 94.2), turned to -90 degrees
- moved J10 13.8 mm to (129.5, 132.5)
- moved J3 3.55 mm to (122.8, 102.2), turned to 90 degrees
- moved J2 3.26 mm to (130.8, 102.2), turned to -90 degrees
- moved J8 1.67 mm to (123.3, 132.5)
- moved C5 1.48 mm to (128.5, 124.8)
- moved A1 1.26 mm to (103.9, 97.2)
- moved J12 1.03 mm to (126.4, 132.5)
- moved C3 0.89 mm to (130.2, 114.2), turned to -90 degrees
- moved J4 0.79 mm to (118.0, 100.2)
- moved C10 0.76 mm to (114.7, 116.5)
- moved Y1 0.76 mm to (112.2, 117.5)
- moved C11 0.76 mm to (114.7, 118.5), turned to -90 degrees
- moved C2 0.76 mm to (127.5, 126.5)
- moved D2 0.60 mm to (70.2, 134.0)
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Routing:
- net GND: track 12.9 -> 106.2 mm, vias 0 -> 41
- net +3.3V: track 12.2 -> 99.3 mm
- net +12V: track 0.00 -> 72.9 mm
- net +5V: track 0.00 -> 54.7 mm
- net /enable_sm: track 0.00 -> 39.9 mm, vias 0 -> 2
- net /step_sm: track 0.00 -> 24.7 mm, vias 0 -> 2
- net /NRST: track 0.00 -> 24.3 mm
- net /dir_sm: track 0.00 -> 21.1 mm, vias 0 -> 2
- net /SERVO4: track 0.00 -> 16.3 mm
- net /SW_DIO: track 0.00 -> 16.1 mm
- net /I2C_SCL: track 0.00 -> 13.7 mm
- net /I2C_SDA: track 0.00 -> 11.7 mm
- net /USART1_TX: track 0.00 -> 11.7 mm
- net /USART1_RX: track 0.00 -> 11.6 mm
- net /SW_CLK: track 0.00 -> 11.6 mm
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- added copper zone on F.Cu, net +3.3V
- added copper zone on F.Cu, net +5V
- added copper zone on F.Cu, net GND

Commit message: -
Parts:
- added G***: LOGO, LOGO, F.Cu at (139.2, 136.0)
- moved C14 21.2 mm to (70.5, 140.0)
- moved J5 1.39 mm to (81.3, 133.5)
- moved D2 0.79 mm to (71.0, 134.2), turned to 0 degrees
- moved SW1 0.34 mm to (122.5, 94.3)
- moved C1 0.25 mm to (115.2, 114.2)
- moved J2 0.25 mm to (131.0, 102.2)
- moved R2 0.25 mm to (132.0, 115.5)
- moved C15 0.15 mm to (79.0, 106.2)
- moved C10 0.10 mm to (114.8, 116.5)
- moved C11 0.10 mm to (114.8, 118.5)
Connections:
- D2 pad 2: +12V -> /DC_IN
- J5 pad 1: +12V -> /DC_IN
Routing:
- net +3.3V: track 99.3 -> 160.6 mm, vias 0 -> 10
- net GND: track 106.2 -> 151.1 mm, vias 41 -> 74
- net +12V: track 72.9 -> 58.4 mm
- net /dir_sm: track 21.1 -> 33.0 mm
- net /step_sm: track 24.7 -> 35.4 mm
- net /DC_IN: track 0.00 -> 7.75 mm
- net /enable_sm: track 39.9 -> 45.3 mm
- net /SW_DIO: track 16.1 -> 17.6 mm
- removed copper zone on F.Cu, net +3.3V
- removed copper zone on F.Cu, net +5V
Other:
- board text added: "-"
- board text added: "0"
- board text added: "1"
- board text added: "2025/12/23 VERSION 1.0"
- board text added: "BOOT"
- board text added: "BUCK CONVERTER"
- board text added: "C13"
- board text added: "J11"
- board text added: "J12"
- board text added: "J7"
- board text added: "J8"
- board text added: "MOTOR DRIVER"
- board text added: "RESET"
- board text added: "RUBIK'S SOLVER V1"
- board text added: "SERVO1"
- board text added: "SERVO2"
- board text added: "SERVO3"
- board text added: "SERVO4"
- board text added: "SERVO5"
- board text added: "STEPPER MOTOR"
- board text added: "SWD"
- board text added: "UART"
- board text added: "USB"

Commit message: -
Parts:
- removed J10, J11, J7, J8: Conn_01x03_Pin, Connector_PinHeader_1.00mm:PinHeader_1x03_P1.00mm_Vertical
- added A2: Pololu_Breakout_A4988, Module:Pololu_Breakout-16_15.2x20.3mm, F.Cu at (103.6, 145.8)
- added C18: 100u, Capacitor_THT:C_Radial_D8.0mm_H7.0mm_P3.50mm, F.Cu at (128.0, 141.8)
- added J16: Conn_01x04_Pin, Connector_PinHeader_1.00mm:PinHeader_1x04_P1.00mm_Vertical, F.Cu at (130.5, 132.5)
- moved D1 9.91 mm to (95.6, 133.9)
- moved C12 9.91 mm to (93.0, 136.7)
- moved C13 9.91 mm to (97.0, 136.7)
- moved R4 9.91 mm to (98.0, 134.1)
- moved U2 9.91 mm to (95.0, 142.2)
- moved G*** 0.79 mm to (139.0, 135.2)
Connections:
- net /dir_sm renamed /dir_sm_1
- net /enable_sm renamed /enable_sm_1
- net /step_sm renamed /step_sm_1
- J12 pad 1: /SERVO5 -> /SERVO1
- U1 pad 21: /SERVO1 -> /enable_sm_2
- U1 pad 22: /SERVO2 -> /step_sm_2
- U1 pad 23: /SERVO3 -> /dir_sm_2
- U1 pad 29: /SERVO5 -> /SERVO1
- U1 pad 42: /SERVO4 -> unconnected-(U1-PA9-Pad42)
Routing:
- net /dir_sm_2: track 0.00 -> 32.7 mm
- net Net-(A2-1B): track 0.00 -> 28.6 mm
- net /step_sm_2: track 0.00 -> 28.6 mm
- net Net-(A2-1A): track 0.00 -> 25.8 mm
- net Net-(A2-2A): track 0.00 -> 23.1 mm
- net Net-(A2-2B): track 0.00 -> 19.6 mm
- net /SERVO4: track 16.3 -> 0.00 mm
- net +3.3V: track 160.6 -> 172.4 mm, vias 10 -> 11
- net /SERVO2: track 9.92 -> 0.00 mm
- net /enable_sm_2: track 0.00 -> 9.09 mm
- net /SERVO5: track 8.87 -> 0.00 mm
- net /SERVO3: track 8.84 -> 0.00 mm
- net GND: track 151.1 -> 158.5 mm
- net +5V: track 54.8 -> 61.8 mm, vias 0 -> 2
- net +12V: track 58.4 -> 65.3 mm
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Other:
- board text added: "RUBIK'S SOLVER V1.1"
- board text removed: "C13"
- board text removed: "J11"
- board text removed: "J7"
- board text removed: "J8"
- board text removed: "RUBIK'S SOLVER V1"
- board text removed: "SERVO1"
- board text removed: "SERVO2"
- board text removed: "SERVO3"
- board text removed: "SERVO4"
- board text removed: "SERVO5"

Commit message: -
Parts:
- moved J9 11.2 mm to (107.0, 97.5), turned to 0 degrees
- moved J14 4.13 mm to (104.5, 110.5)
- moved J6 4.13 mm to (63.5, 110.5)
- moved A1 3.50 mm to (103.9, 93.7)
- moved C15 2.75 mm to (79.0, 103.5)
- moved J12 2.50 mm to (126.5, 130.0)
Routing:
- net +12V: track 65.3 -> 122.1 mm, vias 0 -> 1
- net Net-(A1-2B): track 3.76 -> 18.6 mm
- net Net-(A1-2A): track 3.13 -> 15.7 mm
- net +3.3V: track 172.4 -> 183.8 mm, vias 11 -> 12
- net Net-(A1-1A): track 3.33 -> 13.1 mm
- net GND: track 158.5 -> 149.5 mm
- net Net-(A1-1B): track 4.27 -> 9.87 mm
- net /dir_sm_1: track 33.0 -> 36.6 mm
- net /enable_sm_1: track 45.3 -> 48.8 mm
- net /step_sm_1: track 35.4 -> 38.9 mm
- net +5V: track 61.8 -> 64.5 mm
- net /SERVO1: track 8.87 -> 6.41 mm
- net Net-(A2-1A): track 25.8 -> 24.4 mm
- net Net-(A2-2A): track 23.1 -> 22.0 mm
- net Net-(A2-1B): track 28.6 -> 28.1 mm
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Other:
- board text removed: "STEPPER MOTOR"

Commit message: -
Routing:
- net Net-(A2-1B): track 28.1 -> 27.3 mm
Other:
- board text added: "2025/12/23 VERSION 1.1"
- board text removed: "2025/12/23 VERSION 1.0"
Changed lines of the file:
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@@
 			(usegerberattributes yes)
 			(usegerberadvancedattributes yes)
-			(creategerberjobfile yes)
+			(creategerberjobfile no)
 			(dashed_line_dash_ratio 12.000000)
 			(dashed_line_gap_ratio 3.000000)
@@
 			(outputformat 1)
 			(mirror no)
-			(drillshape 1)
+			(drillshape 0)
 			(scaleselection 1)
-			(outputdirectory "")
+			(outputdirectory "manufacturing/")
 		)
 	)
@@
 		)
 	)
-	(gr_text "2025/12/23\nVERSION 1.0"
+	(gr_text "2025/12/23\nVERSION 1.1"
 		(at 70.5 96.25 0)
 		(layer "F.SilkS")
@@
 	)
 	(segment
-		(start 128 132.5)
-		(end 130.5 132.5)
-		(width 0.5)
-		(layer "F.Cu")
-		(net 73)
-	)
-	(segment
 		(start 123 135.5)
 		(end 125 135.5)
@@
 	)
 	(segment
-		(start 116 142.5)
-		(end 123 135.5)
-		(width 0.5)
+		(start 130.5 132.5)
+		(end 128 132.5)
+		(width 0.3)
 		(layer "F.Cu")
 		(net 73)
 	)
 	(segment
-		(start 130.5 132.5)
-		(end 129.775 132.5)
-		(width 0.3)
+		(start 116 142.5)
+		(end 123 135.5)
+		(width 0.5)
 		(layer "F.Cu")
 		(net 73)
